Commit message: First commit: commiting a first runnable version of google cartographer with ouster Lidar

File: rover_2dnav/cartographer_ros/urdf/os1_lidar.urdf (robot description, URDF)
Before this commit: robot os_sensor, 5 links, 4 joints
Links:
- removed link os_lidar1
- removed link os_lidar2
- added link os
- added link os_lidar; visual cylinder length=0.07 radius=0.05
Joints:
- removed joint os_link_joint1
- removed joint os_link_joint2
- added joint os_link_joint: type fixed, parent os_sensor, child os_lidar, origin xyz=0.0 0.0 0.03618 rpy=0 0 3.14159
- added joint os_link_joint_legacy: type fixed, parent base_link, child os, origin xyz=0.00 0. 0.03618 rpy=0. 0 0

File: rover_2dnav/cartographer_ros/urdf/os1_sensors_test.urdf (robot description, URDF)
Before this commit: robot os_sensor, 5 links, 4 joints
Links:
- added link os_lidar; visual cylinder length=0.07 radius=0.05
- added link os_sensor1
- added link os_sensor2
- link base_link: geometry visual mesh filename=package://rover_2dnav/meshes/Unnamed-Mercedes Benz Sprinter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
Joints:
- added joint os_link_joint: type fixed, parent os_sensor, child os_lidar, origin xyz=0.0 0.0 0.03618 rpy=0 0 3.14159
- added joint sensor_link_joint1: type fixed, parent base_link, child os_sensor1, origin xyz=1.12 -1.1 -0.475856 rpy=0.561937 0.75593 0.07367
- added joint sensor_link_joint2: type fixed, parent base_link, child os_sensor2, origin xyz=1.07831 0.970087 -0.39168 rpy=2.63308 2.39713 3.11967
- joint os_link_joint1: parent os_sensor -> os_sensor1
- joint os_link_joint2: origin xyz=1.12 0.95 0.46 rpy=0.61086 0 3.14159 -> xyz=0.0 0.0 0.03618 rpy=0 0 3.14159; parent os_sensor -> os_sensor2
- joint sensor_link_joint: origin xyz=0 0 0 rpy=0 0 0 -> xyz=0.0 0.0 0.0 rpy=0 0 0
